File: kicad/rc_car/rc_car.kicad_pcb (KiCad board)
At the start: 2 copper layers, 67 x 56.5 mm, 32 parts, among them J1 Raspberry_Pi_2_3, J3 Screw_Terminal_01x02, J4 Conn_01x03_Male, J5 Conn_01x03_Male, J6 Conn_01x03_Male, J7 Conn_01x04_Female, J8 Conn_01x04_Male, Q1 BC547, SW1 SW_Push_Dual, U1 4001

Commit message: [kicad/rc_car] wired pins of the atmega to some connectors
Parts:
- added J3: Conn_01x07_Female, Connector_PinHeader_2.54mm:PinHeader_1x07_P2.54mm_Vertical, F.Cu at (140.5, 82.4)
- added J4: Conn_01x04_Female, Connector_PinHeader_2.54mm:PinHeader_1x04_P2.54mm_Vertical, F.Cu at (161.8, 81.2)
- U1: footprint Package_DIP:DIP-14_W7.62mm_LongPads -> Package_DIP:DIP-14_W7.62mm_Socket_LongPads
- moved A1 0.22 mm to (119.4, 61.5)
- renumbered C8 to C3, C3 to C4, C4 to C5, C5 to C6, J3 to J2, J7 to J5, J4 to J6, J5 to J7, J6 to J8, J8 to J9
Connections:
- A1 pad 10: Net-(A1-Pad10) -> /d7
- A1 pad 11: Net-(A1-Pad11) -> /d8
- A1 pad 19: Net-(A1-Pad19) -> /a0
- A1 pad 20: Net-(A1-Pad20) -> /a1
- A1 pad 21: Net-(A1-Pad21) -> /a2
- A1 pad 22: Net-(A1-Pad22) -> /a3
- A1 pad 5: Net-(A1-Pad5) -> /d2
- A1 pad 6: Net-(A1-Pad6) -> /d3
- A1 pad 7: Net-(A1-Pad7) -> /d4
- A1 pad 8: Net-(A1-Pad8) -> /d5
- A1 pad 9: Net-(A1-Pad9) -> /d6
Routing:
- net /a0: track 0.00 -> 40.8 mm
- net /a1: track 0.00 -> 38.0 mm
- net /d5: track 0.00 -> 37.9 mm
- net /d2: track 0.00 -> 37.5 mm
- net /d4: track 0.00 -> 37.0 mm
- net /d3: track 0.00 -> 36.6 mm
- net /a2: track 0.00 -> 35.1 mm
- net /d6: track 0.00 -> 33.8 mm
- net /a3: track 0.00 -> 32.3 mm
- net /d7: track 0.00 -> 29.9 mm
- net /d8: track 0.00 -> 27.1 mm
- net +7.5V: track 2.51 -> 4.65 mm
- net VCC: track 160.6 -> 158.5 mm
